Commit message: feat(nav+mcu): IRL tuning WIP — scripted drive, dead reckoning odom, gait tweaks
Nav/launch:
- new scripted_cmd_vel node + example yaml + real_scripted_drive.launch.py
- new cmd_vel_restrict and dead_reckoning_odom nodes
- real_object_seek_no_gyro.launch.py variant + updates to real_object_seek/real_slam_raw
- nav2 and slam_toolbox real-robot param tuning
- object_seeker, ball_searcher, scan_tilt_filter refinements

MCU:
- GaitController + GaitRosParticipant updates

Misc:
- docker/Dockerfile, URDF lidar tweak, detection_utils, COMMANDS.md docs

Co-Authored-By: Claude Opus 4.7 <noreply@anthropic.com>

File: ros2_ws/src/seeker_description/urdf/seeker_hexapod.urdf.xacro (robot description, xacro)
@@ -239,5 +239,5 @@
     <parent link="base_link"/>
     <child  link="lidar_link"/>
-    <origin xyz="0 0 ${body_z/2}" rpy="0 0 ${pi}"/>
+    <origin xyz="0 0 ${body_z/2}" rpy="0 0 0"/>
   </joint>
   <!-- Gazebo LiDAR sensor → /gz/scan, bridged to /mcu/scan -->
