Commit message: feat: it is worky now with full integration

File: ros2_ws/src/seeker_description/urdf/seeker_hexapod.urdf.xacro (robot description, xacro)
@@ -93,5 +93,5 @@
       <origin xyz="${mount_x} ${mount_y} 0" rpy="0 0 ${mount_angle}"/>
       <axis xyz="0 0 1"/>
-      <limit lower="${hip_lo}" upper="${hip_hi}" effort="2.0" velocity="3.14"/>
+      <limit lower="${hip_lo}" upper="${hip_hi}" effort="3.0" velocity="3.14"/>
       <dynamics damping="0.1" friction="0.0"/>
     </joint>
@@ -138,5 +138,5 @@
       <origin xyz="${femur_len} 0 ${-coxa_len}" rpy="0 0 0"/>
       <axis xyz="0 -1 0"/>
-      <limit lower="${knee_lo}" upper="${knee_hi}" effort="2.0" velocity="3.14"/>
+      <limit lower="${knee_lo}" upper="${knee_hi}" effort="5.0" velocity="3.14"/>
       <dynamics damping="0.1" friction="0.0"/>
     </joint>
@@ -147,7 +147,7 @@
         <joint_name>leg_${name}_hip_joint</joint_name>
         <topic>/model/seeker/joint/leg_${name}_hip_joint/0/cmd_pos</topic>
-        <p_gain>80</p_gain>
-        <i_gain>0.1</i_gain>
-        <d_gain>20.0</d_gain>
+        <p_gain>200</p_gain>
+        <i_gain>0.2</i_gain>
+        <d_gain>2.0</d_gain>
       </plugin>
     </gazebo>
@@ -158,6 +158,6 @@
         <joint_name>leg_${name}_knee_joint</joint_name>
         <topic>/model/seeker/joint/leg_${name}_knee_joint/0/cmd_pos</topic>
-        <p_gain>80</p_gain>
-        <i_gain>0.1</i_gain>
+        <p_gain>200</p_gain>
+        <i_gain>0.2</i_gain>
         <d_gain>2.0</d_gain>
       </plugin>
@@ -175,6 +175,6 @@
           <contact>
             <ode>
-              <kp>1e3</kp>   <!-- contact stiffness (default 1e15 is too rigid) -->
-              <kd>100</kd>   <!-- contact damping — kd_crit≈26 for kp=1e3; 100 = overdamped -->
+              <kp>1e4</kp>
+              <kd>40</kd>
             </ode>
           </contact>

Commit message: fix(urdf): flip lidar_joint 180° around Z
Match mounted lidar orientation on the real robot; LD14P is installed
facing aft relative to the body frame.

File: ros2_ws/src/seeker_description/urdf/seeker_hexapod.urdf.xacro (robot description, xacro)
@@ -239,5 +239,5 @@
     <parent link="base_link"/>
     <child  link="lidar_link"/>
-    <origin xyz="0 0 ${body_z/2}" rpy="0 0 0"/>
+    <origin xyz="0 0 ${body_z/2}" rpy="0 0 ${pi}"/>
   </joint>
   <!-- Gazebo LiDAR sensor → /gz/scan, bridged to /mcu/scan -->

Commit message: feat: add camera based nav, fix orientations, lidar, other stuff

File: ros2_ws/src/seeker_description/urdf/seeker_hexapod.urdf.xacro (robot description, xacro)
@@ -239,5 +239,8 @@
     <parent link="base_link"/>
     <child  link="lidar_link"/>
-    <origin xyz="0 0 ${body_z/2}" rpy="0 0 0"/>
+    <!-- Physical LD14P is mounted with its 0° mark pointing toward the
+         rear of the chassis, so rotate the LiDAR frame 180° about Z to
+         keep "lidar_link +X" == "base_link forward". -->
+    <origin xyz="0 0 ${body_z/2}" rpy="0 0 ${pi}"/>
   </joint>
   <!-- Gazebo LiDAR sensor → /gz/scan, bridged to /mcu/scan -->
